File: hardware/layout.sch (KiCad schematic)
At the start: 16 parts, among them U1 Arduino_UNO_R3, U1 ME2108

Commit message: Update layout.sch
Parts:
- removed L1: 22uH, symbol Device:L
- removed U?: ~, symbol solar_objects:ME2108A33P
- added C3, C4: .1 uF, symbol Device:C
- gave numbers to parts that had none: 1
Connections:
- net +5V: now also C3.1, C4.2
- net GND: now also C3.2, C4.1
Other:
- company: (none) -> Vedant Misra
- title: (none) -> Portable Solar Powered Charger
